File: Assets/Adafruit feather express/Adafruit Feather STM32F405 Express.kicad_pcb (KiCad board)
At the start: 2 copper layers, 50.8 x 22.9 mm, 63 parts, among them Q3 DMG3405, SW1 KMR2, U1 25Q16, U2 AP2112-3.3, U3 MCP73831T-2ACI/OT, X1 JSTPH, X2 32.768, Y1 12mhz

Commit message: fixed .step file not loading
Parts:
- @HOLE0, @HOLE1: footprint (none) -> Adafruit Feather STM32F405 Express:
Changed lines of the file:
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@@
     )
   )
-  (footprint "" (layer "F.Cu")
+  (footprint "Adafruit Feather STM32F405 Express:" (layer "F.Cu")
     (at 171.3611 113.8936)
     (fp_text reference "@HOLE1" (at 0 0) (layer "F.SilkS") hide
@@
     )
   )
-  (footprint "" (layer "F.Cu")
+  (footprint "Adafruit Feather STM32F405 Express:" (layer "F.Cu")
     (at 171.3611 96.1136)
     (fp_text reference "@HOLE0" (at 0 0) (layer "F.SilkS") hide
@@
     (pad "MT2" smd rect (at 13.6 -14.44 270) (size 1.4 1.9) (layers "B.Cu" "B.Paste" "B.Mask")
       (net 1 "GND") (solder_mask_margin 0.0508) (thermal_bridge_angle 0))
+    (model "${KIPRJMOD}/3dmodels/SD Card.step"
+      (offset (xyz 7 -8.5 0))
+      (scale (xyz 1 1 1))
+      (rotate (xyz 0 -180 -90))
+    )
   )
   (footprint "Adafruit Feather STM32F405 Express:TESTPOINT_ROUND_1.5MM" (layer "B.Cu")
