File: Power Circuit/Power Circuit.kicad_sch (KiCad schematic)
At the start: 13 parts, among them U1 TPS61087DRCT

Commit message: added boost converter
Parts:
- C4, C5: value 47uf -> 10uf
Changed lines of the file:
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@@
       (effects (font (size 1.27 1.27)) (justify left))
     )
-    (property "Value" "47uf" (at 173.99 46.9963 0)
+    (property "Value" "10uf" (at 173.99 46.9963 0)
       (effects (font (size 1.27 1.27)) (justify left))
     )
@@
       (effects (font (size 1.27 1.27)) (justify left))
     )
-    (property "Value" "47uf" (at 184.15 46.9963 0)
-      (effects (font (size 1.27 1.27)) (justify left))
-    )
+    (property "Value" "10uf" (at 184.15 46.9963 0)
+      (effects (font (size 1.27 1.27)) (justify left))
+    )
